Commit message: Added gripper with constant link

File: urdf/ur_macro.xacro (robot description, xacro)
@@ -314,4 +314,19 @@
       </inertial>
     </link>
+    <!-- Custom gripper -->
+    <link name="${tf_prefix}gripper_link">
+      <visual>
+        <origin xyz="0 0 0" rpy="0 0 0"/>
+        <geometry>
+          <box size="0.3 0.4 0.2"/>
+        </geometry>
+      </visual>
+      <collision>
+        <origin xyz="0 0 0" rpy="0 0 0"/>
+        <geometry>
+          <box size="0.3 0.4 0.2"/>
+        </geometry>
+      </collision>
+    </link>
     <!-- base_joint fixes base_link to the environment -->
     <joint name="${tf_prefix}base_joint" type="fixed">
@@ -444,4 +459,10 @@
       <child link="${tf_prefix}tool0"/>
     </joint>
+    <!-- Fixed joint from flange to gripper -->
+    <joint name="${tf_prefix}flange-gripper" type="fixed">
+      <parent link="${tf_prefix}flange" />
+      <child link="${tf_prefix}gripper_link" />
+      <origin xyz="0.5 0 0" rpy="0 0 0"/>
+    </joint>
   </xacro:macro>
 </robot>

Commit message: changed the origin of the box geometry

File: urdf/ur_macro.xacro (robot description, xacro)
@@ -317,13 +317,13 @@
     <link name="${tf_prefix}gripper_link">
       <visual>
+        <origin xyz="0.15 0 0" rpy="0 0 0"/>
+        <geometry>
+          <box size="0.3 0.4 0.2"/>
+        </geometry>
+      </visual>
+      <collision>
         <origin xyz="0 0 0" rpy="0 0 0"/>
         <geometry>
-          <box size="0.3 0.4 0.2"/>
-        </geometry>
-      </visual>
-      <collision>
-        <origin xyz="0 0 0" rpy="0 0 0"/>
-        <geometry>
-          <box size="0.3 0.4 0.2"/>
+          <box size="0.15 0.4 0.2"/>
         </geometry>
       </collision>
@@ -463,5 +463,5 @@
       <parent link="${tf_prefix}flange" />
       <child link="${tf_prefix}gripper_link" />
-      <origin xyz="0.5 0 0" rpy="0 0 0"/>
+      <origin xyz="0.0 0 0" rpy="0 0 0"/>
     </joint>
   </xacro:macro>
